Commit message: Back up rough and flat RL experiments on Test_RL_v2

File: src/nino_description/urdf/nino.urdf.xacro (robot description, xacro)
@@ -29,12 +29,12 @@
   <link name="base_link">
     <inertial>
-      <!-- CAD mass and moments; lateral COM and lateral cross-products are
-           made exactly symmetric so equal wheel commands produce straight travel. -->
+      <!-- CAD center of mass and moments scaled to a 2.5 kg chassis;
+           lateral COM and cross-products stay symmetric. -->
       <origin xyz="0.0592774512 0 0.0848297985" rpy="0 0 0"/>
-      <mass value="3.6594075244"/>
+      <mass value="2.5"/>
       <inertia
-        ixx="0.0286794731" ixy="0" ixz="-0.00039888648"
-        iyy="0.0473970329" iyz="0"
-        izz="0.0716779090"/>
+        ixx="0.0195929757" ixy="0" ixz="-0.0002725076"
+        iyy="0.0323802641" iyz="0"
+        izz="0.0489682473"/>
     </inertial>
     <visual>
@@ -72,7 +72,8 @@
     <inertial>
       <origin xyz="0 0 0" rpy="0 0 0"/>
-      <mass value="0.10"/>
-      <inertia ixx="0.00004" ixy="0" ixz="0"
-               iyy="0.00004" iyz="0" izz="0.00007"/>
+      <mass value="1.3"/>
+      <!-- Solid-cylinder inertia for radius 0.0375 m and height 0.05 m. -->
+      <inertia ixx="0.000727864583" ixy="0" ixz="0"
+               iyy="0.000727864583" iyz="0" izz="0.0009140625"/>
     </inertial>
     <visual>
@@ -93,11 +94,15 @@
     <parent link="base_link"/>
     <child link="laser"/>
-    <origin xyz="0.10 0 0.18" rpy="0 0 0"/>
+    <!-- Center of the four-hole top-plate pattern (x=0.1725/0.2275,
+         y=+/-0.015); the cylinder bottom sits on the z=0.14 plate. -->
+    <origin xyz="0.20 0 0.165" rpy="0 0 0"/>
   </joint>
   <!-- A shallow downward-looking scan gives the policy deployable preview of
        low cables and terrain before the casters reach them. It is mounted
        just beyond the 0.31 m CAD chassis nose so the robot cannot occlude its
-       rays. At 0.2325 m height and 0.45 rad pitch it observes the floor about
-       0.48 m ahead; the horizontal fan distinguishes left/right terrain. -->
+       rays. Its housing sits above the horizontal /scan plane, so the main
+       LiDAR does not mistake this sensor for an obstacle. At 0.2625 m height
+       and 0.45 rad pitch it observes the floor about 0.54 m ahead; the
+       horizontal fan distinguishes left/right terrain. -->
   <link name="terrain_laser">
     <visual>
@@ -109,5 +114,5 @@
     <parent link="base_link"/>
     <child link="terrain_laser"/>
-    <origin xyz="0.33 0 0.17" rpy="0 0.45 0"/>
+    <origin xyz="0.33 0 0.20" rpy="0 0.45 0"/>
   </joint>
   <gazebo reference="terrain_laser">
@@ -222,9 +227,10 @@
       <inertial>
         <origin xyz="0 0 ${com_z}" rpy="0 0 0"/>
-        <mass value="0.4194392311"/>
+        <!-- Keep the CAD inertia ratios when increasing each wheel to 0.8 kg. -->
+        <mass value="0.8"/>
         <inertia
-          ixx="0.00043046655" ixy="0" ixz="0"
-          iyy="0.00043046655" iyz="0"
-          izz="0.00076090197"/>
+          ixx="0.00082103250" ixy="0" ixz="0"
+          iyy="0.00082103250" iyz="0"
+          izz="0.00145127478"/>
       </inertial>
       <visual>

Commit message: Update Governor

File: src/nino_description/urdf/nino.urdf.xacro (robot description, xacro)
@@ -4,4 +4,6 @@
     name="controllers_file"
     default="$(find nino_control)/config/controllers.yaml"/>
+  <xacro:arg name="contact_lab" default="false"/>
+  <xacro:arg name="terrain_preview" default="true"/>
   <!-- Dimensions measured from the supplied SolidWorks STL export. -->
   <xacro:property name="drive_wheel_radius" value="0.0625"/>
@@ -116,4 +118,5 @@
     <origin xyz="0.33 0 0.20" rpy="0 0.45 0"/>
   </joint>
+  <xacro:if value="$(arg terrain_preview)">
   <gazebo reference="terrain_laser">
     <sensor name="terrain_preview_sensor" type="gpu_lidar">
@@ -152,4 +155,5 @@
     </sensor>
   </gazebo>
+  </xacro:if>
   <gazebo>
     <plugin filename="gz-sim-imu-system" name="gz::sim::systems::Imu"/>
@@ -163,4 +167,5 @@
       <odom_frame>world</odom_frame>
       <robot_base_frame>base_footprint</robot_base_frame>
+      <xacro:if value="$(arg contact_lab)"><dimensions>3</dimensions></xacro:if>
       <odom_publish_frequency>50</odom_publish_frequency>
       <odom_topic>/model/nino/odometry</odom_topic>
@@ -332,4 +337,27 @@
   <xacro:caster index="left" y="0.088"/>
   <xacro:caster index="right" y="-0.088"/>
+  <!-- Research-only contact oracle: never connected to deployed governor. -->
+  <xacro:macro name="contact_logger_sensor" params="component link:='' collision:=''">
+    <gazebo reference="${link if link else component+'_link'}">
+      <sensor name="${component}_contact" type="contact">
+        <always_on>true</always_on>
+        <update_rate>100</update_rate>
+        <contact>
+          <collision>${collision if collision else component+'_link_collision'}</collision>
+          <topic>/nino/contact_lab/${component}</topic>
+        </contact>
+      </sensor>
+    </gazebo>
+  </xacro:macro>
+  <xacro:if value="$(arg contact_lab)">
+    <xacro:contact_logger_sensor component="left_wheel"/>
+    <xacro:contact_logger_sensor component="right_wheel"/>
+    <xacro:contact_logger_sensor component="caster_left_wheel"/>
+    <xacro:contact_logger_sensor component="caster_right_wheel"/>
+    <xacro:contact_logger_sensor component="caster_bracket_left"/>
+    <xacro:contact_logger_sensor component="caster_bracket_right"/>
+    <xacro:contact_logger_sensor component="chassis" link="base_footprint"
+      collision="base_footprint_fixed_joint_lump__base_link_collision"/>
+  </xacro:if>
   <!-- Identical contact parameters on the left and right prevent artificial
        yaw.  Caster friction is lower so the swivels align without scrubbing. -->

Commit message: Fix needed

File: src/nino_description/urdf/nino.urdf.xacro (robot description, xacro)
@@ -6,4 +6,5 @@
   <xacro:arg name="contact_lab" default="false"/>
   <xacro:arg name="terrain_preview" default="true"/>
+  <xacro:arg name="caster_wheel_damping" default="0.01"/>
   <!-- Dimensions measured from the supplied SolidWorks STL export. -->
   <xacro:property name="drive_wheel_radius" value="0.0625"/>
@@ -332,5 +333,5 @@
       <axis xyz="0 0 -1"/>
       <limit effort="1.0" velocity="30.0"/>
-      <dynamics damping="0.01" friction="0.0"/>
+      <dynamics damping="$(arg caster_wheel_damping)" friction="0.0"/>
     </joint>
   </xacro:macro>
